Commit message: Half visual size, 5% collision size

File: src/hector_quadrotor/hector_quadrotor_description/urdf/quadrotor_base.urdf.xacro (robot description, xacro)
@@ -20,5 +20,5 @@
         <origin xyz="0 0 0" rpy="0 0 0" />
         <geometry>
-          <mesh filename="package://hector_quadrotor_description/meshes/quadrotor/quadrotor_base.stl"/>
+          <mesh filename="package://hector_quadrotor_description/meshes/quadrotor/quadrotor_base_05.stl"/>
         </geometry>
       </collision>

File: src/hector_quadrotor/hector_quadrotor_description/urdf/quadrotor_with_cam.urdf.xacro (robot description, xacro)
@@ -8,5 +8,5 @@
     <!-- Forward facing camera -->
     <xacro:include filename="$(find hector_sensors_description)/urdf/generic_camera.urdf.xacro" />
-    <xacro:generic_camera name="front_cam" parent="base_link" ros_topic="camera/image" cam_info_topic="camera/camera_info" update_rate="10" res_x="320" res_y="240" image_format="R8G8B8" hfov="90">
+    <xacro:generic_camera name="front_cam" parent="base_link" ros_topic="camera/image" cam_info_topic="camera/camera_info" update_rate="10" res_x="1333" res_y="1000" image_format="R8G8B8" hfov="90">
       <origin xyz="0.05 0.0 -0.06" rpy="0 0 0"/>
     </xacro:generic_camera>

Commit message: Potentially working no ground truth

File: src/hector_quadrotor/hector_quadrotor_description/urdf/quadrotor_base.urdf.xacro (robot description, xacro)
@@ -20,5 +20,5 @@
         <origin xyz="0 0 0" rpy="0 0 0" />
         <geometry>
-          <mesh filename="package://hector_quadrotor_description/meshes/quadrotor/quadrotor_base_05.stl"/>
+          <mesh filename="package://hector_quadrotor_description/meshes/quadrotor/quadrotor_base_half.stl"/>
         </geometry>
       </collision>

Commit message: Likely working without ground truth

File: src/hector_quadrotor/hector_quadrotor_description/urdf/quadrotor_base.urdf.xacro (robot description, xacro)
@@ -20,5 +20,5 @@
         <origin xyz="0 0 0" rpy="0 0 0" />
         <geometry>
-          <mesh filename="package://hector_quadrotor_description/meshes/quadrotor/quadrotor_base_half.stl"/>
+          <mesh filename="package://hector_quadrotor_description/meshes/quadrotor/quadrotor_base_05.stl"/>
         </geometry>
       </collision>

File: src/hector_quadrotor/hector_quadrotor_gazebo/urdf/quadrotor_sensors.gazebo.xacro (robot description, xacro)
@@ -48,5 +48,5 @@
             <velocityGaussianNoise>0.05 0.05 0.05</velocityGaussianNoise>
           </plugin> -->
-          <plugin name="quadrotor_groundtruth_sim" filename="libgazebo_ros_p3d.so">
+          <!-- <plugin name="quadrotor_groundtruth_sim" filename="libgazebo_ros_p3d.so">
             <updateRate>100.0</updateRate>
             <bodyName>base_link</bodyName>
@@ -54,5 +54,5 @@
             <gaussianNoise>0.0</gaussianNoise>
             <frameName>$(arg world_frame)</frameName>
-          </plugin>
+          </plugin> -->
         </gazebo>
   </xacro:macro>

Commit message: updated collision

File: src/hector_quadrotor/hector_quadrotor_description/urdf/quadrotor_base.urdf.xacro (robot description, xacro)
@@ -12,5 +12,5 @@
       </inertial>
       <visual>
-        <origin xyz="0 0 0" rpy="0 0 0" />
+        <origin xyz="0 0 0.091" rpy="0 0 0" />
         <geometry>
           <mesh filename="package://hector_quadrotor_description/meshes/quadrotor/quadrotor_base.dae"/>
@@ -26,5 +26,5 @@
     <!-- Sonar height sensor -->
     <xacro:sonar_sensor name="sonar" parent="base_link" ros_topic="sonar_height" update_rate="10" min_range="0.03" max_range="3.0" field_of_view="${40*pi/180}" ray_count="3">
-      <origin xyz="-0.16 0.0 -0.012" rpy="0 ${90*pi/180} 0"/>
+      <origin xyz="-0.14 0.0 0.09" rpy="0 ${90*pi/180} 0"/>
     </xacro:sonar_sensor>
   </xacro:macro>

File: src/hector_quadrotor/hector_quadrotor_description/urdf/quadrotor_with_2cams.urdf.xacro (robot description, xacro)
@@ -9,10 +9,10 @@
     <xacro:include filename="$(find hector_sensors_description)/urdf/generic_camera.urdf.xacro" />
     <xacro:generic_camera name="front_cam" parent="base_link" ros_topic="camera/image" cam_info_topic="camera/camera_info" update_rate="10" res_x="1333" res_y="1000" image_format="R8G8B8" hfov="90">
-      <origin xyz="0.05 0.0 -0.06" rpy="0 0 0"/>
+      <origin xyz="0.1 0.0 0.075" rpy="0 0 0"/>
     </xacro:generic_camera>
      <!-- Downward facing camera -->
     <xacro:include filename="$(find hector_sensors_description)/urdf/generic_camera.urdf.xacro" />
     <xacro:generic_camera name="downward_cam" parent="base_link" ros_topic="down_camera/image" cam_info_topic="down_camera/camera_info" update_rate="20" res_x="640" res_y="480" image_format="L8" hfov="100">
-      <origin xyz="0.4 0.0 -0.0" rpy="0 ${M_PI/2} 0"/>
+      <origin xyz="0.19 0.0 0.092" rpy="0 ${M_PI/2} 0"/>
     </xacro:generic_camera>
 </robot>

Commit message: New model

File: src/hector_quadrotor/hector_quadrotor_description/urdf/quadrotor_base.urdf.xacro (robot description, xacro)
@@ -14,5 +14,5 @@
         <origin xyz="0 0 0.091" rpy="0 0 0" />
         <geometry>
-          <mesh filename="package://hector_quadrotor_description/meshes/quadrotor/quadrotor_base.dae"/>
+          <mesh filename="package://hector_quadrotor_description/meshes/quadrotor/quadrotor_baseRC.dae"/>
         </geometry>
       </visual>
@@ -20,5 +20,5 @@
         <origin xyz="0 0 0" rpy="0 0 0" />
         <geometry>
-          <mesh filename="package://hector_quadrotor_description/meshes/quadrotor/quadrotor_base_half.stl"/>
+          <mesh filename="package://hector_quadrotor_description/meshes/quadrotor/quadrotor_baseRC.stl"/>
         </geometry>
       </collision>

Commit message: working on customtexture

File: src/hector_quadrotor/hector_quadrotor_description/urdf/quadrotor_base.urdf.xacro (robot description, xacro)
@@ -12,5 +12,5 @@
       </inertial>
       <visual>
-        <origin xyz="0 0 0.091" rpy="0 0 0" />
+        <origin xyz="0 0 0" rpy="0 0 0" />
         <geometry>
           <mesh filename="package://hector_quadrotor_description/meshes/quadrotor/quadrotor_baseRC.dae"/>
@@ -26,5 +26,5 @@
     <!-- Sonar height sensor -->
     <xacro:sonar_sensor name="sonar" parent="base_link" ros_topic="sonar_height" update_rate="10" min_range="0.03" max_range="3.0" field_of_view="${40*pi/180}" ray_count="3">
-      <origin xyz="-0.14 0.0 0.09" rpy="0 ${90*pi/180} 0"/>
+      <origin xyz="-0.05 0.0 -0.005" rpy="0 ${90*pi/180} 0"/>
     </xacro:sonar_sensor>
   </xacro:macro>

File: src/hector_quadrotor/hector_quadrotor_description/urdf/quadrotor_with_5cams.urdf.xacro (robot description, xacro)
@@ -2,4 +2,5 @@
 <robot name="quadrotor" xmlns:xacro="http://www.ros.org/wiki/xacro">
     <xacro:property name="M_PI" value="3.1415926535897931" />
+    <xacro:property name="C_HEIGHT" value="-0.013" />
     <!-- Included URDF Files -->
     <xacro:include filename="$(find hector_quadrotor_description)/urdf/quadrotor_base.urdf.xacro" />
@@ -9,25 +10,25 @@
     <xacro:include filename="$(find hector_sensors_description)/urdf/generic_camera.urdf.xacro" />
     <xacro:generic_camera name="front_cam" parent="base_link" ros_topic="camera/image" cam_info_topic="camera/camera_info" update_rate="10" res_x="1000" res_y="570" image_format="R8G8B8" hfov="120">
-      <origin xyz="0.1 0.0 0.075" rpy="0 0 0"/>
+      <origin xyz="0.1 0.0 ${C_HEIGHT}" rpy="0 0 0"/>
     </xacro:generic_camera>
     <!-- Backwards facing camera -->
     <xacro:include filename="$(find hector_sensors_description)/urdf/generic_camera.urdf.xacro" />
     <xacro:generic_camera name="back_cam" parent="base_link" ros_topic="back_camera/image" cam_info_topic="back_camera/camera_info" update_rate="10" res_x="1000" res_y="570" image_format="R8G8B8" hfov="120">
-      <origin xyz="-0.1 0.0 0.075" rpy="0 0 ${M_PI}"/>
+      <origin xyz="-0.1 0.0 ${C_HEIGHT}" rpy="0 0 ${M_PI}"/>
     </xacro:generic_camera>
     <!-- Left facing camera -->
     <xacro:include filename="$(find hector_sensors_description)/urdf/generic_camera.urdf.xacro" />
     <xacro:generic_camera name="left_cam" parent="base_link" ros_topic="left_camera/image" cam_info_topic="left_camera/camera_info" update_rate="10" res_x="1000" res_y="570" image_format="R8G8B8" hfov="120">
-      <origin xyz="0.0 0.1 0.075" rpy="0 0 ${M_PI/2}"/>
+      <origin xyz="0.0 0.1 ${C_HEIGHT}" rpy="0 0 ${M_PI/2}"/>
     </xacro:generic_camera>
     <!-- Right facing camera -->
     <xacro:include filename="$(find hector_sensors_description)/urdf/generic_camera.urdf.xacro" />
     <xacro:generic_camera name="right_cam" parent="base_link" ros_topic="right_camera/image" cam_info_topic="right_camera/camera_info" update_rate="10" res_x="1000" res_y="570" image_format="R8G8B8" hfov="120">
-      <origin xyz="0.0 -0.1 0.075" rpy="0 0 ${3*M_PI/2}"/>
+      <origin xyz="0.0 -0.1 ${C_HEIGHT}" rpy="0 0 ${3*M_PI/2}"/>
     </xacro:generic_camera>
      <!-- Downward facing camera -->
     <xacro:include filename="$(find hector_sensors_description)/urdf/generic_camera.urdf.xacro" />
     <xacro:generic_camera name="downward_cam" parent="base_link" ros_topic="down_camera/image" cam_info_topic="down_camera/camera_info" update_rate="20" res_x="640" res_y="480" image_format="R8G8B8" hfov="90">
-      <origin xyz="0.19 0.0 0.092" rpy="0 ${M_PI/2} 0"/>
+      <origin xyz="0.0 0.0 ${C_HEIGHT}" rpy="0 ${M_PI/2} 0"/>
     </xacro:generic_camera>
 </robot>
