Commit message: Added rotating camera links

File: src/hector_quadrotor/hector_quadrotor_description/urdf/quadrotor_with_2cams.urdf.xacro (robot description, xacro)
@@ -6,10 +6,27 @@
     <!-- Instantiate quadrotor_base_macro once (has no parameters atm) -->
     <xacro:quadrotor_base_macro />
+    <!-- Add Rotatable Joint for Forward-Facing Camera -->
+    <!-- Rotating base -->
+    <link name="front_cam_base">
+      <inertial>
+        <mass value="0.1"/>
+        <origin xyz="0 0 0"/>
+        <inertia ixx="0.01" ixy="0" ixz="0" iyy="0.01" iyz="0" izz="0.01"/>
+      </inertial>
+    </link>
+    <!-- Rotating joint -->
+    <joint name="rotate_front_cam_joint" type="revolute">
+      <parent link="base_link"/>
+      <child link="front_cam_base"/>
+      <origin xyz="0.1 0.0 0.075" rpy="0 0 0"/> <!-- Match camera origin -->
+      <axis xyz="0 0 1"/> <!-- Rotate around Z-axis -->
+      <limit lower="0.0" upper="6.283185307" effort="1.0" velocity="1.0"/> <!-- 0° to 360° -->
+    </joint>
     <!-- Forward facing camera -->
     <xacro:include filename="$(find hector_sensors_description)/urdf/generic_camera.urdf.xacro" />
-    <xacro:generic_camera name="front_cam" parent="base_link" ros_topic="camera/image" cam_info_topic="camera/camera_info" update_rate="10" res_x="1750" res_y="1000" image_format="R8G8B8" hfov="120">
-      <origin xyz="0.1 0.0 0.075" rpy="0 0 0"/>
+    <xacro:generic_camera name="front_cam" parent="front_cam_base" ros_topic="camera/image" cam_info_topic="camera/camera_info" update_rate="10" res_x="1750" res_y="1000" image_format="R8G8B8" hfov="120">
+      <origin xyz="0 0 0" rpy="0 0 0"/> <!-- Origin now relative to front_cam_base -->
     </xacro:generic_camera>
-     <!-- Downward facing camera -->
+    <!-- Downward facing camera -->
     <xacro:include filename="$(find hector_sensors_description)/urdf/generic_camera.urdf.xacro" />
     <xacro:generic_camera name="downward_cam" parent="base_link" ros_topic="down_camera/image" cam_info_topic="down_camera/camera_info" update_rate="20" res_x="640" res_y="480" image_format="R8G8B8" hfov="90">

Commit message: 5 cameras

File: src/hector_quadrotor/hector_quadrotor_description/urdf/quadrotor_with_2cams.urdf.xacro (robot description, xacro)
@@ -11,4 +11,19 @@
       <origin xyz="0.1 0.0 0.075" rpy="0 0 0"/>
     </xacro:generic_camera>
+    <!-- Backwards facing camera -->
+    <xacro:include filename="$(find hector_sensors_description)/urdf/generic_camera.urdf.xacro" />
+    <xacro:generic_camera name="back_cam" parent="base_link" ros_topic="back_camera/image" cam_info_topic="back_camera/camera_info" update_rate="10" res_x="1750" res_y="1000" image_format="R8G8B8" hfov="120">
+      <origin xyz="-0.1 0.0 0.075" rpy="0 0 ${M_PI}"/>
+    </xacro:generic_camera>
+    <!-- Left facing camera -->
+    <xacro:include filename="$(find hector_sensors_description)/urdf/generic_camera.urdf.xacro" />
+    <xacro:generic_camera name="left_cam" parent="base_link" ros_topic="left_camera/image" cam_info_topic="left_camera/camera_info" update_rate="10" res_x="1750" res_y="1000" image_format="R8G8B8" hfov="120">
+      <origin xyz="0.0 0.1 0.075" rpy="0 0 ${M_PI/2}"/>
+    </xacro:generic_camera>
+    <!-- Right facing camera -->
+    <xacro:include filename="$(find hector_sensors_description)/urdf/generic_camera.urdf.xacro" />
+    <xacro:generic_camera name="right_cam" parent="base_link" ros_topic="right_camera/image" cam_info_topic="right_camera/camera_info" update_rate="10" res_x="1750" res_y="1000" image_format="R8G8B8" hfov="120">
+      <origin xyz="0.0 -0.1 0.075" rpy="0 0 ${3*M_PI/2}"/>
+    </xacro:generic_camera>
      <!-- Downward facing camera -->
     <xacro:include filename="$(find hector_sensors_description)/urdf/generic_camera.urdf.xacro" />

Commit message: PID implementation

File: src/hector_quadrotor/hector_quadrotor_description/urdf/quadrotor_with_2cams.urdf.xacro (robot description, xacro)
@@ -12,19 +12,4 @@
       <origin xyz="0.1 0.0 ${C_HEIGHT}" rpy="0 0 0"/>
     </xacro:generic_camera>
-    <!-- Backwards facing camera -->
-    <xacro:include filename="$(find hector_sensors_description)/urdf/generic_camera.urdf.xacro" />
-    <xacro:generic_camera name="back_cam" parent="base_link" ros_topic="back_camera/image" cam_info_topic="back_camera/camera_info" update_rate="10" res_x="1000" res_y="570" image_format="R8G8B8" hfov="120">
-      <origin xyz="-0.1 0.0 ${C_HEIGHT}" rpy="0 0 ${M_PI}"/>
-    </xacro:generic_camera>
-    <!-- Left facing camera -->
-    <xacro:include filename="$(find hector_sensors_description)/urdf/generic_camera.urdf.xacro" />
-    <xacro:generic_camera name="left_cam" parent="base_link" ros_topic="left_camera/image" cam_info_topic="left_camera/camera_info" update_rate="10" res_x="1000" res_y="570" image_format="R8G8B8" hfov="120">
-      <origin xyz="0.0 0.1 ${C_HEIGHT}" rpy="0 0 ${M_PI/2}"/>
-    </xacro:generic_camera>
-    <!-- Right facing camera -->
-    <xacro:include filename="$(find hector_sensors_description)/urdf/generic_camera.urdf.xacro" />
-    <xacro:generic_camera name="right_cam" parent="base_link" ros_topic="right_camera/image" cam_info_topic="right_camera/camera_info" update_rate="10" res_x="1000" res_y="570" image_format="R8G8B8" hfov="120">
-      <origin xyz="0.0 -0.1 ${C_HEIGHT}" rpy="0 0 ${3*M_PI/2}"/>
-    </xacro:generic_camera>
      <!-- Downward facing camera -->
     <xacro:include filename="$(find hector_sensors_description)/urdf/generic_camera.urdf.xacro" />
