Commit message: Fixed collisions

File: src/hector_quadrotor/hector_quadrotor_description/urdf/quadrotor_with_5cams.urdf.xacro (robot description, xacro)
@@ -2,5 +2,5 @@
 <robot name="quadrotor" xmlns:xacro="http://www.ros.org/wiki/xacro">
     <xacro:property name="M_PI" value="3.1415926535897931" />
-    <xacro:property name="C_HEIGHT" value="-0.013" />
+    <xacro:property name="C_HEIGHT" value="-0.0152" />
     <!-- Included URDF Files -->
     <xacro:include filename="$(find hector_quadrotor_description)/urdf/quadrotor_base.urdf.xacro" />

Commit message: Consistent first sign

File: src/hector_quadrotor/hector_quadrotor_description/urdf/quadrotor_with_5cams.urdf.xacro (robot description, xacro)
@@ -10,20 +10,20 @@
     <xacro:include filename="$(find hector_sensors_description)/urdf/generic_camera.urdf.xacro" />
     <xacro:generic_camera name="front_cam" parent="base_link" ros_topic="camera/image" cam_info_topic="camera/camera_info" update_rate="10" res_x="1000" res_y="570" image_format="R8G8B8" hfov="120">
-      <origin xyz="0.1 0.0 ${C_HEIGHT}" rpy="0 0 0"/>
+      <origin xyz="0.1 0.0 ${C_HEIGHT}" rpy="0 0.15 0"/>
     </xacro:generic_camera>
     <!-- Backwards facing camera -->
     <xacro:include filename="$(find hector_sensors_description)/urdf/generic_camera.urdf.xacro" />
     <xacro:generic_camera name="back_cam" parent="base_link" ros_topic="back_camera/image" cam_info_topic="back_camera/camera_info" update_rate="10" res_x="1000" res_y="570" image_format="R8G8B8" hfov="120">
-      <origin xyz="-0.1 0.0 ${C_HEIGHT}" rpy="0 0 ${M_PI}"/>
+      <origin xyz="-0.1 0.0 ${C_HEIGHT}" rpy="0 0.15 ${M_PI}"/>
     </xacro:generic_camera>
     <!-- Left facing camera -->
     <xacro:include filename="$(find hector_sensors_description)/urdf/generic_camera.urdf.xacro" />
     <xacro:generic_camera name="left_cam" parent="base_link" ros_topic="left_camera/image" cam_info_topic="left_camera/camera_info" update_rate="10" res_x="1000" res_y="570" image_format="R8G8B8" hfov="120">
-      <origin xyz="0.0 0.1 ${C_HEIGHT}" rpy="0 0 ${M_PI/2}"/>
+      <origin xyz="0.0 0.1 ${C_HEIGHT}" rpy="0 0.15 ${M_PI/2}"/>
     </xacro:generic_camera>
     <!-- Right facing camera -->
     <xacro:include filename="$(find hector_sensors_description)/urdf/generic_camera.urdf.xacro" />
     <xacro:generic_camera name="right_cam" parent="base_link" ros_topic="right_camera/image" cam_info_topic="right_camera/camera_info" update_rate="10" res_x="1000" res_y="570" image_format="R8G8B8" hfov="120">
-      <origin xyz="0.0 -0.1 ${C_HEIGHT}" rpy="0 0 ${3*M_PI/2}"/>
+      <origin xyz="0.0 -0.1 ${C_HEIGHT}" rpy="0 0.15 ${3*M_PI/2}"/>
     </xacro:generic_camera>
      <!-- Downward facing camera -->

Commit message: PID better

File: src/hector_quadrotor/hector_quadrotor_description/urdf/quadrotor_with_5cams.urdf.xacro (robot description, xacro)
@@ -29,6 +29,6 @@
      <!-- Downward facing camera -->
     <xacro:include filename="$(find hector_sensors_description)/urdf/generic_camera.urdf.xacro" />
-    <xacro:generic_camera name="downward_cam" parent="base_link" ros_topic="down_camera/image" cam_info_topic="down_camera/camera_info" update_rate="20" res_x="640" res_y="480" image_format="R8G8B8" hfov="90">
-      <origin xyz="0.0 0.0 ${C_HEIGHT}" rpy="0 ${M_PI/2} 0"/>
+    <xacro:generic_camera name="downward_cam" parent="base_link" ros_topic="down_camera/image" cam_info_topic="down_camera/camera_info" update_rate="20" res_x="640" res_y="480" image_format="R8G8B8" hfov="150">
+      <origin xyz="0.0 0.0 ${C_HEIGHT-0.05}" rpy="0 ${M_PI/2} 0"/>
     </xacro:generic_camera>
 </robot>
