Commit message: Failed simpler camera custom plugin

File: src/hector_models/hector_sensors_description/urdf/generic_camera.urdf.xacro (robot description, xacro)
@@ -2,5 +2,5 @@
 <robot xmlns:xacro="http://ros.org/wiki/xacro">
   <xacro:property name="M_PI" value="3.1415926535897931" />
-  <xacro:macro name="generic_camera" params="name parent *origin ros_topic cam_info_topic update_rate res_x res_y image_format hfov">
+  <xacro:macro name="generic_camera" params="name parent *origin ros_topic update_rate res_x res_y image_format hfov">
     <joint name="${name}_joint" type="fixed">
       <xacro:insert_block name="origin" />
@@ -51,9 +51,7 @@
           </clip>
         </camera>
-        <plugin name="${name}_camera_controller" filename="libgazebo_ros_camera.so">
-          <cameraName>${name}</cameraName>
+        <!-- Use the custom plugin -->
+        <plugin name="${name}_custom_camera_plugin" filename="libcustom_camera_plugin.so">
           <imageTopicName>${ros_topic}</imageTopicName>
-          <cameraInfoTopicName>${cam_info_topic}</cameraInfoTopicName>
-          <frameName>${name}_optical_frame</frameName>
         </plugin>
       </sensor>

File: src/hector_quadrotor/hector_quadrotor_description/urdf/quadrotor_with_5cams.urdf.xacro (robot description, xacro)
@@ -9,25 +9,25 @@
     <!-- Forward facing camera -->
     <xacro:include filename="$(find hector_sensors_description)/urdf/generic_camera.urdf.xacro" />
-    <xacro:generic_camera name="front_cam" parent="base_link" ros_topic="camera/image" cam_info_topic="camera/camera_info" update_rate="10" res_x="1000" res_y="570" image_format="R8G8B8" hfov="120">
+    <xacro:generic_camera name="front_cam" parent="base_link" ros_topic="camera/image" update_rate="10" res_x="1000" res_y="570" image_format="R8G8B8" hfov="120">
       <origin xyz="0.1 0.0 ${C_HEIGHT}" rpy="0 0 0"/>
     </xacro:generic_camera>
     <!-- Backwards facing camera -->
     <xacro:include filename="$(find hector_sensors_description)/urdf/generic_camera.urdf.xacro" />
-    <xacro:generic_camera name="back_cam" parent="base_link" ros_topic="back_camera/image" cam_info_topic="back_camera/camera_info" update_rate="10" res_x="1000" res_y="570" image_format="R8G8B8" hfov="120">
+    <xacro:generic_camera name="back_cam" parent="base_link" ros_topic="back_camera/image" update_rate="10" res_x="1000" res_y="570" image_format="R8G8B8" hfov="120">
       <origin xyz="-0.1 0.0 ${C_HEIGHT}" rpy="0 0 ${M_PI}"/>
     </xacro:generic_camera>
     <!-- Left facing camera -->
     <xacro:include filename="$(find hector_sensors_description)/urdf/generic_camera.urdf.xacro" />
-    <xacro:generic_camera name="left_cam" parent="base_link" ros_topic="left_camera/image" cam_info_topic="left_camera/camera_info" update_rate="10" res_x="1000" res_y="570" image_format="R8G8B8" hfov="120">
+    <xacro:generic_camera name="left_cam" parent="base_link" ros_topic="left_camera/image" update_rate="10" res_x="1000" res_y="570" image_format="R8G8B8" hfov="120">
       <origin xyz="0.0 0.1 ${C_HEIGHT}" rpy="0 0 ${M_PI/2}"/>
     </xacro:generic_camera>
     <!-- Right facing camera -->
     <xacro:include filename="$(find hector_sensors_description)/urdf/generic_camera.urdf.xacro" />
-    <xacro:generic_camera name="right_cam" parent="base_link" ros_topic="right_camera/image" cam_info_topic="right_camera/camera_info" update_rate="10" res_x="1000" res_y="570" image_format="R8G8B8" hfov="120">
+    <xacro:generic_camera name="right_cam" parent="base_link" ros_topic="right_camera/image" update_rate="10" res_x="1000" res_y="570" image_format="R8G8B8" hfov="120">
       <origin xyz="0.0 -0.1 ${C_HEIGHT}" rpy="0 0 ${3*M_PI/2}"/>
     </xacro:generic_camera>
      <!-- Downward facing camera -->
     <xacro:include filename="$(find hector_sensors_description)/urdf/generic_camera.urdf.xacro" />
-    <xacro:generic_camera name="downward_cam" parent="base_link" ros_topic="down_camera/image" cam_info_topic="down_camera/camera_info" update_rate="20" res_x="640" res_y="480" image_format="R8G8B8" hfov="90">
+    <xacro:generic_camera name="downward_cam" parent="base_link" ros_topic="down_camera/image" update_rate="20" res_x="640" res_y="480" image_format="R8G8B8" hfov="90">
       <origin xyz="0.0 0.0 ${C_HEIGHT}" rpy="0 ${M_PI/2} 0"/>
     </xacro:generic_camera>
